Commit message: xacro issue fixed

File: urdf/pioneer3dx_wheel.xacro (robot description, xacro)
@@ -6,7 +6,7 @@
   xmlns:xacro="http://ros.org/wiki/xacro"
   >
-  <!--<include filename="$(find pioneer)/defs/materials.xacro"/>-->
+  <!--<xacro:include filename="$(find pioneer)/defs/materials.xacro"/>-->
   <!-- Properties (Constants) -->
-  <property name="M_PI" value="3.14159"/>
+  <xacro:property name="M_PI" value="3.14159"/>
 <!-- Right/Left Hubcap + Wheel -->
 <xacro:macro name="p3dx_wheel" params="suffix parent reflect">
